File: civic_serializer/civic_serializer.kicad_sch (KiCad schematic)
At the start: 2 parts, among them IC1 DS90UB925QSQX_NOPB, J1 GPIO

Commit message: - routed part of schematic
Parts:
- added C1, C2, C3: 10u, Capacitor_SMD:C_0805_2012Metric_Pad1.18x1.45mm_HandSolder, symbol Device:C
- added C10, C11, C12: 100n, Capacitor_SMD:C_0805_2012Metric_Pad1.18x1.45mm_HandSolder, symbol Device:C
- added C4, C5, C6, C7, C8, C9: 4.7u, Capacitor_SMD:C_0805_2012Metric_Pad1.18x1.45mm_HandSolder, symbol Device:C
- added D1: LED, LED_SMD:LED_0805_2012Metric_Pad1.15x1.40mm_HandSolder, symbol Device:LED
- added FB1, FB2: FerriteBead, Inductor_SMD:L_0805_2012Metric_Pad1.05x1.20mm_HandSolder, symbol Device:FerriteBead
- added Q1: MMBT2222A, Package_TO_SOT_SMD:SOT-23, symbol Transistor_BJT:MMBT2222A
- added R1: 100R, Resistor_SMD:R_0805_2012Metric_Pad1.20x1.40mm_HandSolder, symbol Device:R
- added R2: 1K, Resistor_SMD:R_0805_2012Metric_Pad1.20x1.40mm_HandSolder, symbol Device:R
- added R3, R4: 0R, Resistor_SMD:R_0805_2012Metric_Pad1.20x1.40mm_HandSolder, symbol Device:R
- added R5: 4K7, Resistor_SMD:R_0805_2012Metric_Pad1.20x1.40mm_HandSolder, symbol Device:R
- added U1: AMS1117-3.3, Package_TO_SOT_SMD:SOT-223-3_TabPin2, symbol Regulator_Linear:AMS1117-3.3
Connections:
- net CLK is gone; now on net PCLK: J1.27 (Pin_27)
- net +5V: now also C1.1, U1.3 (VI)
- net B0: now also IC1.43 (GPO_REG4_/_B0_/_DIN16)
- net B1: now also IC1.44 (I2S_DB_/_GPO_REG5_/_B1_/_DIN17)
- net B2: now also IC1.45 (B2_/_DIN18)
- net B3: now also IC1.46 (B3_/_DIN19)
- net B4: now also IC1.47 (B4_/_DIN20)
- net B5: now also IC1.48 (B5_/_DIN21)
- net B6: now also IC1.1 (B6_/_DIN22)
- net B7: now also IC1.2 (B7_/_DIN23)
- net G0: now also IC1.35 (DIN8_/_G0_/GPIO2)
- net G1: now also IC1.36 (DIN9/G1_/_GPIO3)
- net G2: now also IC1.37 (G2_/_DIN10)
- net G3: now also IC1.38 (G3_/_DIN11)
- net G4: now also IC1.39 (G4_/_DIN12)
- net G5: now also IC1.40 (G5_/_DIN13)
- net G6: now also IC1.41 (G6_/_DIN14)
- net G7: now also IC1.42 (G7_/_DIN15)
- net GND: now also IC1.15 (RES0), C1.2, C12.2, C2.2, C3.2, C4.2, C5.2, C6.2, C7.2, C8.2, C9.2, D1.1 (K), Q1.2 (E), U1.1 (GND)
- net HSYNC: now also IC1.3 (HS)
- net R0: now also IC1.25 (DIN0/_R0/_GPIO0)
- net R1: now also IC1.26 (DIN1_/_R1_/_GPIO1)
- net R2: now also IC1.27 (DIN2/R2)
- net R3: now also IC1.28 (DIN3/R3)
- net R4: now also IC1.29 (DIN4_/_R4)
- net R5: now also IC1.32 (DIN5/R5)
- net R6: now also IC1.33 (DIN6/R6)
- net R7: now also IC1.34 (DIN7/R7)
- net VSYNC: now also IC1.4 (VS)
- net PCLK: now reaches IC1.10 (PCLK)
- net CAPP12: now reaches IC1.14 (CAPP12)
- net CAPP12: now also C6.1
- net CAPHS12: now reaches IC1.17 (CAPHS12)
- net CAPHS12: now also C9.1
- net DOUT-: now reaches IC1.19 (DOUT-)
- net DOUT-: now also C10.1
- net DOUT+: now reaches IC1.20 (DOUT+)
- net DOUT+: now also C11.1
- net VDD33: now reaches IC1.22 (VDD33)
- net VDD33: now also C4.1, FB2.2
- net CMF: now reaches IC1.23 (CMF)
- net CMF: now also C12.1
- net MODE_SEL: now reaches IC1.24 (MODE_SEL)
- net VDDIO: now reaches IC1.30 (VDDIO)
- net VDDIO: now also C5.1, FB1.2
- net DE: now reaches IC1.5 (DE)
- net DE: now also R3.1, R4.1
- net IDX: now reaches IC1.6 (IDX)
- net CAPL12: now reaches IC1.7 (CAPL12)
- net CAPL12: now also C7.1, C8.1
- net SCL: now reaches IC1.8 (SCL)
- net SDA: now reaches IC1.9 (SDA)
- net DEN renamed EN
- net EN: now also R1.1, R4.2
- new net: D1.2 (A), R5.1
- new net: Q1.1 (B), R1.2
- new net 3V3: C2.1, C3.1, FB1.1, FB2.1, R2.2, R5.2, U1.2 (VO)
- new net LVDS+: C11.2
- new net LVDS-: C10.2
- new net NEN: Q1.3 (C), R2.1, R3.2
Other:
- note added: "Inverted and non inverted logic for EN To be selected NEN or DEN"
- note removed: "Additional pin functions: https://pinout.xyz/"
- moved on the sheet: IC1

Commit message: - finished part of the schematic
Parts:
- added C13: 10uF, Capacitor_SMD:C_0805_2012Metric_Pad1.18x1.45mm_HandSolder, symbol Device:C
- added R10, R11, R6, R7: 100R, Resistor_SMD:R_0805_2012Metric_Pad1.20x1.40mm_HandSolder, symbol Device:R
- added R12, R8, R9: 4K7, Resistor_SMD:R_0805_2012Metric_Pad1.20x1.40mm_HandSolder, symbol Device:R
- added R13: 10K, Resistor_SMD:R_0805_2012Metric_Pad1.20x1.40mm_HandSolder, symbol Device:R
Connections:
- net GND: now also C13.2, R11.1, R7.1
- net IDX: now also R10.1, R11.2
- net MODE_SEL: now also R6.1, R7.2
- net SCL: now also R8.1
- net SDA: now also R9.1
- net VDDIO: now also R10.2, R12.2, R13.2, R6.2, R8.2, R9.2
- net PBD: now reaches IC1.21 (PDB)
- net PBD: now also C13.1, R13.1
- net INTB: now reaches IC1.31 (INTB)
- net INTB: now also R12.1

Commit message: - schematic finished
Parts:
- removed Q1: MMBT2222A, Package_TO_SOT_SMD:SOT-23, symbol Transistor_BJT:MMBT2222A
- removed R1: 100R, Resistor_SMD:R_0805_2012Metric_Pad1.20x1.40mm_HandSolder, symbol Device:R
- removed R2: 1K, Resistor_SMD:R_0805_2012Metric_Pad1.20x1.40mm_HandSolder, symbol Device:R
- removed R3, R4: 0R, Resistor_SMD:R_0805_2012Metric_Pad1.20x1.40mm_HandSolder, symbol Device:R
- added I2C: Conn_01x02_Socket, Connector_PinSocket_2.54mm:PinSocket_1x02_P2.54mm_Vertical, symbol Connector:Conn_01x02_Socket
- added LVDS: Conn_01x03_Pin, Connector_JST:JST_NV_B03P-NV_1x03_P5.00mm_Vertical, symbol Connector:Conn_01x03_Pin
- added RV1, RV2: R_Potentiometer_Trim, Potentiometer_THT:Potentiometer_Vishay_T93YA_Vertical, symbol Device:R_Potentiometer_Trim
- R10, R11: now not fitted
- R6, R7: value 100R -> R; now not fitted
Connections:
- net EN is gone; now on net DE: J1.28 (Pin_28)
- net GND: now also IC1.18 (RES1), IC1.49 (EP), LVDS.2 (Pin_2), RV1.3, RV2.3
- net IDX: now also RV2.2
- net LVDS+: now also C10.2, LVDS.3 (Pin_3); no longer C11.2
- net LVDS-: now also C11.2, LVDS.1 (Pin_1); no longer C10.2
- net MODE_SEL: now also RV1.2
- net SCL: now also I2C.1 (Pin_1)
- net SDA: now also I2C.2 (Pin_2)
- net VDDIO: now also RV1.1, RV2.1
- net DOUT+: no longer names the net of IC1.20 (DOUT+)
- net DOUT+: now also C10.1; no longer C11.1
- net DOUT-: no longer names the net of IC1.19 (DOUT-)
- net DOUT-: now also C11.1; no longer C10.1
Other:
- note removed: "Inverted and non inverted logic for EN To be selected NEN or DEN"
- moved on the sheet: C1, C10, C11, C12, C13, C2, C3, C4, C5, C6, C7, C8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

Commit message: - done some of the layout
Parts:
- renumbered C12 to C1, C6 to C10, C10 to C11, C11 to C12, C1 to C2, C2 to C3, C3 to C4, C4 to C6, C9 to C7, C7 to C8, C8 to C9, I2C to I2C1, LVDS to LVDS1, R5 to R1, R13 to R2, R12 to R3, R8 to R4, R9 to R5, R10 to R6, R6 to R7, R11 to R8, R7 to R9, RV2 to RV1, RV1 to RV2

Commit message: - layout finished
Parts:
- added IDX2, MDE1: TestPoint, Connector_PinSocket_2.54mm:PinSocket_1x01_P2.54mm_Vertical, symbol Connector:TestPoint
- C1, C10, C11, C12, C13, C5, C6, C7, C8, C9: footprint Capacitor_SMD:C_0805_2012Metric_Pad1.18x1.45mm_HandSolder -> Capacitor_SMD:C_0603_1608Metric_Pad1.08x0.95mm_HandSolder
- FB1, FB2: footprint Inductor_SMD:L_0805_2012Metric_Pad1.05x1.20mm_HandSolder -> Inductor_SMD:L_0603_1608Metric_Pad1.05x0.95mm_HandSolder
- R2, R3, R4, R5, R6, R7, R8, R9: footprint Resistor_SMD:R_0805_2012Metric_Pad1.20x1.40mm_HandSolder -> Resistor_SMD:R_0603_1608Metric_Pad0.98x0.95mm_HandSolder
- renumbered D1 to 5V1, RV1 to IDX1, RV2 to MD_SEL1
Connections:
- net IDX: now also IDX2.1
- net MODE_SEL: now also MDE1.1
- net DOUT+: now reaches C11.1, IC1.20 (DOUT+)
- net DOUT-: now reaches C12.1, IC1.19 (DOUT-)
