File: civic_serializer/civic_serializer.kicad_pcb (KiCad board)
At the start: 2 copper layers, 65 x 30 mm, 38 parts, among them IC1 DS90UB925QSQX_NOPB, J1 GPIO, U1 AMS1117-3.3

Commit message: - minor lvds trace lenght matching - added generated gerber files
Parts:
- moved C12 0.89 mm to (153.3, 85.6)
- moved C11 0.38 mm to (153.3, 84.1)
- moved MD_SEL1 0.13 mm to (126.3, 94.9)
Routing:
- net LVDS-: track 7.04 -> 7.99 mm
Other:
- board text added: "+"
- board text added: "-"
- board text added: "117 @2025"
- board text added: "5V"
- board text added: "IDX"
- board text added: "LVDS"
- board text added: "MDE"
- board text added: "Video Serializer"

Commit message: - updated vias dimensions - regenerated gerbers
Routing:
- net G4: track 28.4 -> 33.1 mm
- net B7: track 37.2 -> 39.0 mm
- net B4: track 26.7 -> 28.3 mm
- net GND: track 81.0 -> 82.6 mm, vias 10 -> 11
- net MODE_SEL: track 48.4 -> 50.0 mm
- net R4: track 32.2 -> 30.7 mm, vias 0 -> 1
- net B6: track 29.7 -> 31.1 mm
- net B3: track 25.9 -> 27.3 mm
- net DE: track 44.9 -> 43.8 mm
- net G0: track 18.3 -> 19.2 mm
- net G1: track 16.9 -> 17.8 mm
- net B2: track 30.5 -> 31.4 mm
- net B5: track 30.8 -> 31.7 mm
- net VDDIO: track 97.9 -> 98.7 mm
- net R5: track 21.0 -> 21.5 mm
